Commit message: Added urdfs, edited them, and verified with rviz.

File: urdf/beer_rothaus/beer_rothaus.urdf (robot description, URDF)
Before this commit: robot my_object, 1 links, 0 joints
Links:
- added link grasp_loc; visual sphere radius=0.05
Joints:
- added joint grasp_loc_joint: type fixed, parent base_link, child grasp_loc, origin xyz=0 0 0 rpy=0 0 0

File: urdf/robot/aslaug0.urdf (robot description, URDF)
Before this commit: robot panda, 14 links, 13 joints
Links:
- link base_link: geometry collision mesh filename=package://aslaug/../../../../aslaug3d_simulation/urdf/robot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; collision mesh filename=package://aslaug/../../../../aslaug3d_simulation/urdf/robot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
- link front_laser: geometry collision box size=0.05 0.05 0.07; visual mesh filename=package://aslaug/../../../../aslaug3d_simulation/urdf/robot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
- link panda_hand: geometry collision mesh filename=package://aslaug/../../../../aslaug3d_simulation/urdf/robot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; visual mesh filename=package://aslaug/../../../../aslaug3d_simulation/urdf/robot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
- link panda_link0: geometry collision mesh filename=package://aslaug/../../../../aslaug3d_simulation/urdf/robot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; visual mesh filename=package://aslaug/../../../../aslaug3d_simulation/urdf/robot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
- link panda_link1: geometry collision mesh filename=package://aslaug/../../../../aslaug3d_simulation/urdf/robot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; visual mesh filename=package://aslaug/../../../../aslaug3d_simulation/urdf/robot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
- link panda_link2: geometry collision mesh filename=package://aslaug/../../../../aslaug3d_simulation/urdf/robot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; visual mesh filename=package://aslaug/../../../../aslaug3d_simulation/urdf/robot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
- link panda_link3: geometry collision mesh filename=package://aslaug/../../../../aslaug3d_simulation/urdf/robot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; visual mesh filename=package://aslaug/../../../../aslaug3d_simulation/urdf/robot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
- link panda_link4: geometry collision mesh filename=package://aslaug/../../../../aslaug3d_simulation/urdf/robot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; visual mesh filename=package://aslaug/../../../../aslaug3d_simulation/urdf/robot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
- link panda_link5: geometry collision mesh filename=package://aslaug/../../../../aslaug3d_simulation/urdf/robot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; visual mesh filename=package://aslaug/../../../../aslaug3d_simulation/urdf/robot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
- link panda_link6: geometry collision mesh filename=package://aslaug/../../../../aslaug3d_simulation/urdf/robot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; visual mesh filename=package://aslaug/../../../../aslaug3d_simulation/urdf/robot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
- link panda_link7: geometry collision mesh filename=package://aslaug/../../../../aslaug3d_simulation/urdf/robot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; visual mesh filename=package://aslaug/../../../../aslaug3d_simulation/urdf/robot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

Commit message: Updated colors of URDFs

File: urdf/beer_rothaus/beer_rothaus.urdf (robot description, URDF)
Before this commit: robot my_object, 2 links, 1 joints
Links:
- link grasp_loc: geometry visual sphere radius=0.035

File: urdf/robot/aslaug.urdf (robot description, URDF)
Before this commit: robot panda, 14 links, 13 joints
Links:
- added link rear_laser, mass 0.130; collision box size=0.05 0.05 0.07; visual mesh filename=meshes/ust-10lx.stl
Joints:
- added joint rear_laser_joint: type fixed, parent base_link, child rear_laser, origin xyz=-0.3932 0 0.2330 rpy=0 0 3.141592

Commit message: Removed collision from setpoint which was grinding our gears

File: urdf/beer_rothaus/beer_rothaus.urdf (robot description, URDF)
Before this commit: robot my_object, 2 links, 1 joints
Links:
- link base_link: geometry visual mesh filename=beer_rothaus.dae
