Commit message: Post paper

File: urdf/human/leg1.urdf (robot description, URDF)
Before this commit: robot human_leg, 1 links, 0 joints
Links:
- added link body, mass 10.0; collision cylinder length=0.8 radius=0.25; visual cylinder length=0.8 radius=0.25
- link base_link: geometry collision cylinder length=0.5 radius=0.055; visual cylinder length=0.5 radius=0.055
Joints:
- added joint leg_to_body: type fixed, parent base_link, child body, origin xyz=0 0 0.9 rpy=0 0 0
